File: bridge/bridge.kicad_pcb (KiCad board)
At the start: 2 copper layers, 29 parts, among them J1 Screw_Terminal_01x02, J2 Screw_Terminal_01x02, J3 Screw_Terminal_01x02, J4 Screw_Terminal_01x03, Q1 STGP7NC60HD, Q2 STGP7NC60HD, Q3 STGP7NC60HD, Q4 STGP7NC60HD

Commit message: fix bridge, still figuring out layout
Parts:
- added H1: MountingHole_Pad, MountingHole:MountingHole_3.2mm_M3_Pad_Via, F.Cu at (29.0, 24.0)
- added H2: MountingHole_Pad, MountingHole:MountingHole_3.2mm_M3_Pad_Via, F.Cu at (121.0, 24.0)
- added H3: MountingHole_Pad, MountingHole:MountingHole_3.2mm_M3_Pad_Via, F.Cu at (121.0, 116.0)
- added H4: MountingHole_Pad, MountingHole:MountingHole_3.2mm_M3_Pad_Via, F.Cu at (29.0, 116.0)
- added H5: MountingHole_Pad, MountingHole:MountingHole_3.2mm_M3_Pad_Via, F.Cu at (19.4, 3.48)
- added H6: MountingHole_Pad, MountingHole:MountingHole_3.2mm_M3_Pad_Via, F.Cu at (19.4, 11.4)
- added J5: Conn_01x01_Pin, conn:TE_1217861-1, B.Cu at (31.0, 59.0)
- added T1: P0584NL, footprints:P0584NL_PUL, F.Cu at (40.8, 71.4)
- added T2: P0584NL, footprints:P0584NL_PUL, F.Cu at (40.8, 87.4)
- D1, D2, D3, D4, D5, D6, D7, D8, J1, J2, R1, R2, R3, R4, R5: moved to B.Cu
- J3: value Screw_Terminal_01x02 -> Conn_01x01_Pin; footprint conn:PHOENIX_1935161 -> conn:TE_1217861-1; moved to B.Cu
- moved J1 171.9 mm to (31.0, 103.0), turned to -90 degrees
- moved C2 169.5 mm to (32.0, 53.2), turned to 90 degrees
- moved J2 165.5 mm to (39.0, 114.0)
- moved D1 161.9 mm to (55.0, 102.0), turned to 90 degrees
- moved J3 160.2 mm to (31.0, 93.0)
- moved D3 160.1 mm to (49.0, 101.0), turned to 180 degrees
- moved D2 144.0 mm to (73.0, 102.5), turned to 90 degrees
- moved D4 142.7 mm to (66.5, 101.5), turned to 180 degrees
- moved R6 128.0 mm to (71.2, 55.0)
- moved D7 124.0 mm to (88.0, 106.0), turned to 180 degrees
- moved R3 113.8 mm to (31.0, 88.7), turned to 90 degrees
- moved D8 104.3 mm to (108.0, 105.0), turned to 180 degrees
- moved C5 81.6 mm to (98.0, 39.0), turned to 180 degrees
- moved C3 80.6 mm to (118.0, 53.2), turned to 90 degrees
- moved R1 64.5 mm to (58.5, 102.0), turned to -90 degrees
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Connections:
- net GDT4B renamed GDT4A
- C1 pad 1: GDT2A -> GDT2B
- C2 pad 2: GDT2A -> GDT2B
- C3 pad 2: GDT2A -> GDT2B
- C4 pad 2: GDT2A -> GDT2B
- C5 pad 2: GDT2A -> GDT2B
- D2 pad 1: GDT2B -> GDT2A
- D4 pad 2: GDT2A -> GDT2B
- D8 pad 2: GDT2A -> GDT2B
- D9 pad -: GDT2A -> GDT2B
- J1 pad 1: GDT1B -> Net-(J1-Pin_1)
- J1 pad 2: GDT1A -> Net-(J1-Pin_2)
- J2 pad 1: GDT2B -> Net-(J2-Pin_1)
- J2 pad 2: GDT2A -> Net-(J2-Pin_2)
- Q2 pad 3: GDT2A -> GDT2B
- Q4 pad 3: GDT2A -> GDT2B
- R2 pad 2: GDT2B -> GDT2A
- R6 pad 2: GDT2A -> GDT2B
Routing:
- net Net-(D9-PadAC2): track 0.00 -> 29.7 mm
- net NTRL: track 0.00 -> 28.8 mm
- net HOT: track 0.00 -> 16.4 mm
- net Earth: track 0.00 -> 14.6 mm
- net Net-(D2-A): track 0.00 -> 0.85 mm
- net Net-(D1-A): track 0.00 -> 0.85 mm
- added copper zone on F.Cu, net GDT2B
- added copper zone on B.Cu, net Net-(Q1-C)
Other:
- board outline added: 100 x 100 mm
